File: XY/BusProtection.kicad_sch (KiCad schematic)
At the start: 72 parts, among them Q1 NX3008NBKS, Q10 MBT2222ADW1T1, Q11 NX3008NBKS, Q12 MBT2222ADW1T1, Q13 NX3008NBKS, Q14 MBT2222ADW1T1, Q15 NX3008NBKS, Q16 MBT2222ADW1T1, Q2 MBT2222ADW1T1, Q3 NX3008NBKS, Q4 MBT2222ADW1T1, Q5 NX3008NBKS, Q6 MBT2222ADW1T1, Q7 NX3008NBKS, Q8 MBT2222ADW1T1, Q9 NX3008NBKS

Commit message: Updated XY boards
Parts:
- removed C26, C27: 10nF, Capacitor_SMD:C_0603_1608Metric, symbol Device:C
- removed Q5, Q7: NX3008NBKS, Package_TO_SOT_SMD:SOT-363_SC-70-6, symbol mainboard:NX3008NBKS
- removed Q6, Q8: MBT2222ADW1T1, Package_TO_SOT_SMD:SOT-363_SC-70-6, symbol Transistor_BJT:MBT2222ADW1T1
- removed R48, R53: 680R, Resistor_SMD:R_0603_1608Metric, symbol Device:R_Small
- removed R49, R54: 100K, Resistor_SMD:R_0603_1608Metric, symbol Device:R_Small
- removed R50, R51, R55, R56: 10K, Resistor_SMD:R_0603_1608Metric, symbol Device:R_Small
- removed R52, R57: 200K, Resistor_SMD:R_0603_1608Metric, symbol Device:R_Small
- removed R85, R86: DNI (0R), Resistor_SMD:R_0603_1608Metric, symbol Device:R_Small
Other:
- note removed: "Coil Power Jumpers"
- note removed: "I2C Bus Protection - Coil Power Monitor"
