File: XY/I2CDevices.kicad_sch (KiCad schematic)
At the start: 32 parts, among them U1 OPT4003DNPRQ1, U10 NCV891330PD50R2G, U2 ADM1176-1ARMZ-R7, U5 DRV8830DRC, U6 ADM1176-1ARMZ-R7

Commit message: Updated XY boards
Parts:
- removed C22: 3.3nF, Capacitor_SMD:C_0603_1608Metric, symbol Device:C_Small
- removed C23: 0.1uF, Capacitor_SMD:C_0402_1005Metric, symbol Device:C_Small
- removed C28: 0.1uF, Capacitor_SMD:C_0805_2012Metric, symbol Device:C_Small
- removed C34: 1uF, Capacitor_SMD:C_0805_2012Metric, symbol Device:C_Small
- removed C35: 4.7uF, Capacitor_SMD:C_1210_3225Metric, symbol Device:C_Small
- removed C36, C37, C39: 0.1uF, Capacitor_SMD:C_0603_1608Metric, symbol Device:C_Small
- removed C38, C40, C41: 10uF, Capacitor_SMD:C_1206_3216Metric, symbol Device:C_Small
- removed D10: NRVB440MFS, SolarPanels:NRVB440MFSWFT1G, symbol Device:D_Schottky_Small
- removed D9: BAS16HT1G, Diode_SMD:D_SOD-323, symbol Device:D_Small
- removed FL1: SRF2012, SolarPanels:SRF2012, symbol Device:Filter_EMI_CommonMode
- removed L4: XGL3520-222, SolarPanels:XGL3520, symbol Device:L_Small
- removed R32: ?R, Resistor_SMD:R_2512_6332Metric, symbol Device:R_Small
- removed R33: 1K, Resistor_SMD:R_0603_1608Metric, symbol Device:R_Small
- removed R34, R35: 0R, Resistor_SMD:R_0402_1005Metric, symbol Device:R_Small
- removed R60: 0R, Resistor_SMD:R_0603_1608Metric, symbol Device:R_US
- removed R87: 10K, Resistor_SMD:R_0603_1608Metric, symbol Device:R_Small
- removed R94, R95, R96: 0R, Resistor_SMD:R_0603_1608Metric, symbol Device:R_Small
- removed U1: OPT4003DNPRQ1, SolarPanels:OPT4003, symbol SolarPanels:OPT4003DNPRQ1
- removed U10: NCV891330PD50R2G, Package_SO:SOIC-8-1EP_3.9x4.9mm_P1.27mm_EP2.514x3.2mm, symbol SolarPanels:NCV891330PD50R2G
- removed U2: ADM1176-1ARMZ-R7, Package_SO:MSOP-10_3x3mm_P0.5mm, symbol Mainboard:ADM1176-1ARMZ-R7
- removed U5: DRV8830DRC, Package_SON:VSON-10-1EP_3x3mm_P0.5mm_EP1.65x2.4mm, symbol mainboard:DRV8830DRC
- added R90, R91, R92, R93: 0R, Resistor_SMD:R_0603_1608Metric, symbol Device:R_Small
Connections:
- net 3.3V: now also R90.2, R92.2
- net GND: now also R91.1, R93.1
- net A0_S: now reaches U6.8 (A0)
- net A0_S: now also R90.1, R91.2
- net A1_S: now reaches U6.9 (A1)
- net A1_S: now also R92.1, R93.2
- no-connect marks 6 -> 1
Other:
- note removed: "Coil Driver Power Monitor"
- note removed: "Current Limiting Resistor < 1 Ohm"
- note removed: "I2C ADDR 0x64 Install R96: 0x63"
- note removed: "I2C ADDR 0x84 Install R94: 0x80"
- note removed: "I2C ADDR Install R34: 0x45 Install R35: 0x44"
- moved on the sheet: C29, R61, R62, U6
