File: XY/MPPT.kicad_sch (KiCad schematic)
At the start: 15 parts, among them U4 LTC3130

Commit message: Updated XY boards
Parts:
- renumbered C20 to C10, C56 to C11, C21 to C12, C15 to C4, C16 to C5, C53 to C6, C17 to C7, C18 to C8, C19 to C9, L3 to L1, R22 to R1, R23 to R2, R27 to R3, R24 to R4, U4 to U10
Connections:
- net VIN: no longer U10.4 (RUN)
- new net RUN: U10.4 (RUN)
